Commit message: moveit gripper real working

File: robotiq_2f_model/model/robotiq_2f_85.urdf.xacro (robot description, xacro)
@@ -245,5 +245,5 @@
 			<child link="${name}_left_driver"/>
 			<axis xyz="1 0 0"/>
-			<limit lower="${0 * 3.141592 / 180}" upper="${41 * 3.141592 / 180}" effort="176" velocity="${110 * 3.141592 / 180}" />
+			<limit lower="${0 * 3.141592 / 180}" upper="${50 * pi / 180}" effort="176" velocity="${110 * 3.141592 / 180}" />
 			<xacro:unless value="${adaptive_transmission}">
 			<mimic joint="${name}_right_driver_joint" multiplier="1"/>
