Commit message: Fix joint state offset

File: robotiq_description/urdf/robotiq_2f_140/robotiq_2f_140.urdf.xacro (robot description, xacro)
@@ -159,4 +159,7 @@
   </link>
 </xacro:macro>
+<xacro:macro name="fingerpad" params="prefix fingerprefix">
+  <link name="${prefix}${fingerprefix}fingerpad"/>
+</xacro:macro>
 <xacro:macro name="inner_knuckle_joint" params="prefix fingerprefix reflect">
   <joint name="${prefix}${fingerprefix}inner_knuckle_joint" type="revolute">
@@ -211,4 +214,11 @@
     <parent link="${prefix}${fingerprefix}inner_finger" />
     <child link="${prefix}${fingerprefix}fingertip" />
+  </joint>
+</xacro:macro>
+<xacro:macro name="fingerpad_joint" params="prefix fingerprefix">
+  <joint name="${prefix}${fingerprefix}fingerpad_joint" type="fixed">
+    <origin xyz="0 0.0068 0" rpy="0 0 0" />
+    <parent link="${prefix}${fingerprefix}fingertip" />
+    <child link="${prefix}${fingerprefix}fingerpad" />
   </joint>
 </xacro:macro>
@@ -253,4 +263,5 @@
   <xacro:inner_finger prefix="${prefix}" fingerprefix="left_" />
   <xacro:fingertip prefix="${prefix}" fingerprefix="left_" />
+  <xacro:fingerpad prefix="${prefix}" fingerprefix="left_" />
   <xacro:left_outer_knuckle_joint prefix="${prefix}" />
   <xacro:inner_knuckle_joint prefix="${prefix}" fingerprefix="left_" reflect="-1" />
@@ -258,4 +269,5 @@
   <xacro:inner_finger_joint prefix="${prefix}" fingerprefix="left_" />
   <xacro:fingertip_joint prefix="${prefix}" fingerprefix="left_" />
+  <xacro:fingerpad_joint prefix="${prefix}" fingerprefix="left_" />
   <!-- Right gripper link/joints -->
   <xacro:outer_knuckle prefix="${prefix}" fingerprefix="right_" />
@@ -264,4 +276,5 @@
   <xacro:inner_finger prefix="${prefix}" fingerprefix="right_" />
   <xacro:fingertip prefix="${prefix}" fingerprefix="right_" />
+  <xacro:fingerpad prefix="${prefix}" fingerprefix="right_" />
   <xacro:right_outer_knuckle_joint prefix="${prefix}" />
   <xacro:outer_finger_joint prefix="${prefix}" fingerprefix="right_" />
@@ -269,4 +282,5 @@
   <xacro:inner_finger_joint prefix="${prefix}" fingerprefix="right_" />
   <xacro:fingertip_joint prefix="${prefix}" fingerprefix="right_" />
+  <xacro:fingerpad_joint prefix="${prefix}" fingerprefix="right_" />
 </xacro:macro>
 </robot>

Commit message: Updated max limit joint

File: robotiq_description/urdf/robotiq_2f_140/robotiq_2f_140.urdf.xacro (robot description, xacro)
@@ -178,5 +178,5 @@
     <child link="${prefix}left_outer_knuckle" />
     <axis xyz="0 0 1" />
-    <limit lower="0" upper="0.792" velocity="2.0" effort="176" />
+    <limit lower="0" upper="0.786522656" velocity="2.0" effort="176" />
   </joint>
 </xacro:macro>
