Commit message: refactor

File: robotiq_description/urdf/robotiq_ft_300/robotiq_ft_300.urdf.xacro (robot description, xacro)
@@ -36,4 +36,10 @@
     <child link="${prefix}top_link" />
   </joint>
+  <link name="${prefix}reference_frame" />
+  <joint name="${prefix}reference_frame_joint" type="fixed">
+    <origin xyz="0 0 0" rpy="${-pi/2} 0 ${-pi/2}" />
+    <parent link="${prefix}top_link" />
+    <child link="${prefix}reference_frame" />
+  </joint>
 </xacro:macro>
 </robot>
